File: weight_scale.kicad_sch (KiCad schematic)
At the start: 9 parts, among them U1 NAU7802SGI

Commit message: ADD: Terminado la fuente de 24V a 5V, terminado los pines del veronte y tambien el circuito de I2C
Connections:
- net GND: no longer U1.8 (AVSS), U1.9 (DVSS)
- new net EX-: U1.8 (AVSS), U1.9 (DVSS)
Changed lines of the file:
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@@
+	(wire
+		(pts
+			(xy 173.99 96.52) (xy 173.99 99.06)
+		)
+		(stroke
+			(width 0)
+			(type default)
+		)
+	)
 	(wire
 		(pts
@@
 	(symbol
 		(lib_id "power:GND")
-		(at 173.99 99.06 90)
-		(unit 1)
-		(exclude_from_sim no)
-		(in_bom yes)
-		(on_board yes)
-		(dnp no)
-		(fields_autoplaced yes)
-		(property "Reference" "#PWR038"
-			(at 180.34 99.06 0)
-			(effects
-				(font
-					(size 1.27 1.27)
-				)
-				(hide yes)
-			)
-		)
-		(property "Value" "GND"
-			(at 177.8 99.0599 90)
-			(effects
-				(font
-					(size 1.27 1.27)
-				)
-				(justify right)
-			)
-		)
-		(property "Footprint" ""
-			(at 173.99 99.06 0)
-			(effects
-				(font
-					(size 1.27 1.27)
-				)
-				(hide yes)
-			)
-		)
-		(property "Datasheet" ""
-			(at 173.99 99.06 0)
-			(effects
-				(font
-					(size 1.27 1.27)
-				)
-				(hide yes)
-			)
-		)
-		(property "Description" "Power symbol creates a global label with name \"GND\" , ground"
-			(at 173.99 99.06 0)
-			(effects
-				(font
-					(size 1.27 1.27)
-				)
-				(hide yes)
-			)
-		)
-		(pin "1"
-		)
-		(instances
-			(project "pdb"
-				(path "/402e9eb5-eedc-44fb-9e44-3f0a74044b6b/dde71b53-dd0d-4394-ba9e-b4ab950951f7"
-					(reference "#PWR038")
-					(unit 1)
-				)
-			)
-		)
-	)
-	(symbol
-		(lib_id "power:GND")
 		(at 199.39 68.58 90)
 		(unit 1)
@@
 					(unit 1)
 				)
-			)
-		)
-	)
-	(symbol
-		(lib_id "power:GND")
-		(at 173.99 96.52 90)
-		(unit 1)
-		(exclude_from_sim no)
-		(in_bom yes)
-		(on_board yes)
-		(dnp no)
-		(fields_autoplaced yes)
-		(property "Reference" "#PWR041"
-			(at 180.34 96.52 0)
-			(effects
-				(font
-					(size 1.27 1.27)
-				)
-				(hide yes)
-			)
-		)
-		(property "Value" "GND"
-			(at 177.8 96.5199 90)
-			(effects
-				(font
-					(size 1.27 1.27)
-				)
-				(justify right)
-			)
-		)
-		(property "Footprint" ""
-			(at 173.99 96.52 0)
-			(effects
-				(font
-					(size 1.27 1.27)
-				)
-				(hide yes)
-			)
-		)
-		(property "Datasheet" ""
-			(at 173.99 96.52 0)
-			(effects
-				(font
-					(size 1.27 1.27)
-				)
-				(hide yes)
-			)
-		)
-		(property "Description" "Power symbol creates a global label with name \"GND\" , ground"
-			(at 173.99 96.52 0)
-			(effects
-				(font
-					(size 1.27 1.27)
-				)
-				(hide yes)
-			)
-		)
-		(pin "1"
-		)
-		(instances
-			(project "pdb"
-				(path "/402e9eb5-eedc-44fb-9e44-3f0a74044b6b/dde71b53-dd0d-4394-ba9e-b4ab950951f7"
-					(reference "#PWR041")
-					(unit 1)
-				)

Commit message: Primer sesion de ruteo
Parts:
- renumbered C4 to C1, C3 to C2, C1 to C3, C2 to C4, R1 to R3, R2 to R4
Connections:
- net VDD: now reaches C1.1, U1.15 (DVDD)
Changed lines of the file:
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@@
 	(paper "A4")
+	(junction
+		(at 149.86 55.88)
+		(diameter 0)
+		(color 0 0 0 0)
+	)
 	(junction
 		(at 118.11 81.28)
@@
 	)
 	(junction
-		(at 171.45 99.06)
+		(at 176.53 68.58)
 		(diameter 0)
 		(color 0 0 0 0)
 	)
 	(junction
-		(at 149.86 55.88)
-		(diameter 0)
-		(color 0 0 0 0)
-	)
-	(junction
-		(at 186.69 68.58)
+		(at 171.45 99.06)
 		(diameter 0)
 		(color 0 0 0 0)
@@
 	)
 	(junction
+		(at 168.91 62.23)
+		(diameter 0)
+		(color 0 0 0 0)
+	)
+	(junction
 		(at 121.92 73.66)
 		(diameter 0)
 		(color 0 0 0 0)
 	)
+	(junction
+		(at 171.45 68.58)
+		(diameter 0)
+		(color 0 0 0 0)
+	)
 	(no_connect
 		(at 168.91 91.44)
@@
 	(wire
 		(pts
+			(xy 176.53 68.58) (xy 189.23 68.58)
+		)
+		(stroke
+			(width 0)
+			(type default)
+		)
+	)
+	(wire
+		(pts
 			(xy 173.99 96.52) (xy 173.99 99.06)
 		)
@@
 	(wire
 		(pts
+			(xy 171.45 68.58) (xy 176.53 68.58)
+		)
+		(stroke
+			(width 0)
+			(type default)
+		)
+	)
+	(wire
+		(pts
 			(xy 133.35 76.2) (xy 121.92 76.2)
 		)
@@
 	(wire
 		(pts
+			(xy 171.45 55.88) (xy 171.45 68.58)
+		)
+		(stroke
+			(width 0)
+			(type default)
+		)
+	)
+	(wire
+		(pts
 			(xy 125.73 88.9) (xy 118.11 88.9)
 		)
@@
 	(wire
 		(pts
-			(xy 186.69 68.58) (xy 189.23 68.58)
-		)
-		(stroke
-			(width 0)
-			(type default)
-		)
-	)
-	(wire
-		(pts
 			(xy 114.3 81.28) (xy 118.11 81.28)
 		)
@@
 	(wire
 		(pts
-			(xy 168.91 68.58) (xy 186.69 68.58)
-		)
-		(stroke
-			(width 0)
-			(type default)
-		)
-	)
-	(wire
-		(pts
-			(xy 186.69 55.88) (xy 149.86 55.88)
+			(xy 168.91 48.26) (xy 168.91 62.23)
+		)
+		(stroke
+			(width 0)
+			(type default)
+		)
+	)
+	(wire
+		(pts
+			(xy 168.91 68.58) (xy 171.45 68.58)
+		)
+		(stroke
+			(width 0)
+			(type default)
+		)
+	)
+	(wire
+		(pts
+			(xy 149.86 55.88) (xy 171.45 55.88)
 		)
 		(stroke
@@
 		(pts
 			(xy 133.35 100.33) (xy 133.35 91.44)
-		)
-		(stroke
-			(width 0)
-			(type default)
-		)
-	)
-	(wire
-		(pts
-			(xy 186.69 68.58) (xy 186.69 55.88)
 		)
 		(stroke
@@
 			)
 			(justify right)
+		)
+	)
+	(hierarchical_label "VDD"
+		(shape output)
+		(at 168.91 48.26 90)
+		(effects
+			(font
+				(size 1.27 1.27)
+			)
+			(justify left)
 		)
 	)
@@
 		(dnp no)
 		(fields_autoplaced yes)
-		(property "Reference" "#PWR036"
+		(property "Reference" "#PWR053"
 			(at 114.3 73.66 0)
 			(effects
@@
 			(project ""
 				(path "/402e9eb5-eedc-44fb-9e44-3f0a74044b6b/dde71b53-dd0d-4394-ba9e-b4ab950951f7"
-					(reference "#PWR036")
+					(reference "#PWR053")
 					(unit 1)
 				)
@@
 		(on_board yes)
 		(dnp no)
-		(property "Reference" "R1"
+		(property "Reference" "R3"
 			(at 110.49 81.28 90)
 			(effects
@@
 			(project ""
 				(path "/402e9eb5-eedc-44fb-9e44-3f0a74044b6b/dde71b53-dd0d-4394-ba9e-b4ab950951f7"
-					(reference "R1")
+					(reference "R3")
+					(unit 1)
+				)
+			)
+		)
+	)
+	(symbol
+		(lib_id "power:PWR_FLAG")
+		(at 176.53 68.58 0)
+		(unit 1)
+		(exclude_from_sim no)
+		(in_bom yes)
+		(on_board yes)
+		(dnp no)
+		(property "Reference" "#FLG07"
+			(at 176.53 66.675 0)
+			(effects
+				(font
+					(size 1.27 1.27)
+				)
+				(hide yes)
+			)
+		)
+		(property "Value" "PWR_FLAG"
+			(at 182.372 66.802 0)
+			(effects
+				(font
+					(size 1.27 1.27)
+				)
+			)
+		)
+		(property "Footprint" ""
+			(at 176.53 68.58 0)
+			(effects
+				(font
+					(size 1.27 1.27)
+				)
+				(hide yes)
+			)
+		)
+		(property "Datasheet" "~"
+			(at 176.53 68.58 0)
+			(effects
+				(font
+					(size 1.27 1.27)
+				)
+				(hide yes)
+			)
+		)
+		(property "Description" "Special symbol for telling ERC where power comes from"
+			(at 176.53 68.58 0)
+			(effects
+				(font
+					(size 1.27 1.27)
+				)
+				(hide yes)
+			)
+		)
+		(pin "1"
+		)
+		(instances
+			(project ""
+				(path "/402e9eb5-eedc-44fb-9e44-3f0a74044b6b/dde71b53-dd0d-4394-ba9e-b4ab950951f7"
+					(reference "#FLG07")
 					(unit 1)
 				)
@@
 		(dnp no)
 		(fields_autoplaced yes)
-		(property "Reference" "C1"
+		(property "Reference" "C3"
 			(at 127 66.04 90)
 			(effects
@@
 			(project ""
 				(path "/402e9eb5-eedc-44fb-9e44-3f0a74044b6b/dde71b53-dd0d-4394-ba9e-b4ab950951f7"
-					(reference "C1")
+					(reference "C3")
 					(unit 1)
 				)
@@
 		(on_board yes)
 		(dnp no)
-		(property "Reference" "#PWR040"
+		(property "Reference" "#PWR051"
 			(at 187.96 62.23 0)
 			(effects
@@
 			(project "pdb"
 				(path "/402e9eb5-eedc-44fb-9e44-3f0a74044b6b/dde71b53-dd0d-4394-ba9e-b4ab950951f7"
-					(reference "#PWR040")
+					(reference "#PWR051")
 					(unit 1)
 				)
@@
 		(dnp no)
 		(fields_autoplaced yes)
-		(property "Reference" "#PWR037"
+		(property "Reference" "#PWR052"
 			(at 205.74 68.58 0)
 			(effects
@@
 			(project ""
 				(path "/402e9eb5-eedc-44fb-9e44-3f0a74044b6b/dde71b53-dd0d-4394-ba9e-b4ab950951f7"
-					(reference "#PWR037")
+					(reference "#PWR052")
 					(unit 1)
 				)
@@
 		(on_board yes)
 		(dnp no)
-		(property "Reference" "C3"
+		(property "Reference" "C2"
 			(at 196.342 67.056 90)
 			(effects
@@
 			(project "pdb"
 				(path "/402e9eb5-eedc-44fb-9e44-3f0a74044b6b/dde71b53-dd0d-4394-ba9e-b4ab950951f7"
-					(reference "C3")
+					(reference "C2")
 					(unit 1)
 				)
@@
 		(dnp no)
 		(fields_autoplaced yes)
-		(property "Reference" "#PWR039"
+		(property "Reference" "#PWR054"
 			(at 191.77 76.2 0)
 			(effects
@@
 			(project "pdb"
 				(path "/402e9eb5-eedc-44fb-9e44-3f0a74044b6b/dde71b53-dd0d-4394-ba9e-b4ab950951f7"
-					(reference "#PWR039")
+					(reference "#PWR054")
 					(unit 1)
 				)
@@
 		(on_board yes)
 		(dnp no)
-		(property "Reference" "C2"
+		(property "Reference" "C4"
 			(at 180.594 72.136 90)
 			(effects
@@
 			(project "pdb"
 				(path "/402e9eb5-eedc-44fb-9e44-3f0a74044b6b/dde71b53-dd0d-4394-ba9e-b4ab950951f7"
-					(reference "C2")
+					(reference "C4")
 					(unit 1)
 				)
@@
 		(on_board yes)
 		(dnp no)
-		(property "Reference" "C4"
-			(at 172.466 57.15 90)
+		(property "Reference" "C1"
+			(at 177.8 54.356 90)
 			(effects
 				(font
@@
 		)
 		(property "Value" "1uF 50V X7R"
-			(at 172.974 59.182 90)
+			(at 178.308 56.388 90)
 			(effects
 				(font
@@
 			(project "pdb"
 				(path "/402e9eb5-eedc-44fb-9e44-3f0a74044b6b/dde71b53-dd0d-4394-ba9e-b4ab950951f7"
-					(reference "C4")
+					(reference "C1")
 					(unit 1)
 				)
@@
 		(on_board yes)
 		(dnp no)
-		(property "Reference" "R2"
+		(property "Reference" "R4"
 			(at 110.49 88.9 90)
 			(effects
@@
 			(project "pdb"
 				(path "/402e9eb5-eedc-44fb-9e44-3f0a74044b6b/dde71b53-dd0d-4394-ba9e-b4ab950951f7"
-					(reference "R2")
+					(reference "R4")
 					(unit 1)
 				)
