File: pdb.kicad_pcb (KiCad board)
At the start: 4 copper layers, 0 parts

Commit message: Esquematico casi terminado falta agregar el veronte
Parts:
- added C1: 100nF 50V X7R, Capacitor_SMD:C_0603_1608Metric, F.Cu at (131.7, 81.1)
- added C10: 80uF 100V, Capacitor_SMD:CP_Elec_10x10.5, F.Cu at (105.2, 97.5)
- added C11: 68uF 50V, Capacitor_SMD:CP_Elec_6.3x7.7, F.Cu at (103.0, 107.6)
- added C12: 22uF 50V X7R, Capacitor_SMD:C_1812_4532Metric, F.Cu at (121.5, 94.0)
- added C13: 22uF 50V X7R, Capacitor_SMD:C_1812_4532Metric, F.Cu at (121.5, 98.9)
- added C14: 56pF 100V C0G, Capacitor_SMD:C_0603_1608Metric, F.Cu at (125.6, 105.1)
- added C15: 3.3nF 100V C0G, Capacitor_SMD:C_1206_3216Metric, F.Cu at (120.8, 109.8)
- added C2: 100nF 50V X7R, Capacitor_SMD:C_0603_1608Metric, F.Cu at (131.7, 83.6)
- added C3: 1uF 50V X7R, Capacitor_SMD:C_0603_1608Metric, F.Cu at (131.7, 86.1)
- added C4: 1uF 50V X7R, Capacitor_SMD:C_0603_1608Metric, F.Cu at (131.7, 88.6)
- added C5: 1nF 50V C0G, Capacitor_SMD:C_0603_1608Metric, F.Cu at (131.7, 91.1)
- added C6: 100nF 50V C0G, Capacitor_SMD:C_1206_3216Metric, F.Cu at (136.6, 93.1)
- added C7: 2.2nF 50V X7R, Capacitor_SMD:C_0603_1608Metric, F.Cu at (125.6, 102.6)
- added C8: 2.2µF X7R 100V, Capacitor_SMD:C_1206_3216Metric, F.Cu at (120.8, 103.0)
- added C9: 2.2µF X7R 100V, Capacitor_SMD:C_1206_3216Metric, F.Cu at (120.8, 106.4)
- added D1: MBR8H120PC, Library:TO-277C, F.Cu at (124.6, 84.0)
- added F1: Fuse, Library:FUSE-HOLDER XFCN XF-008, F.Cu at (122.1, 70.9)
- added J1: Amass Elec AS150UPW(2+4), Library:CONN-TH_AS150UPW, F.Cu at (65.2, 85.8)
- added J10: BOOMELE 4.2-2*4AW, Connector_Molex:Molex_Mini-Fit_Jr_5569-08A2_2x04_P4.20mm_Horizontal, F.Cu at (161.3, 44.8)
- added J11: MOLEX 39301240, Connector_Molex:Molex_Mini-Fit_Jr_5569-24A2_2x12_P4.20mm_Horizontal, F.Cu at (227.0, 115.2)
- added J12: BOOMELE 4.2-2*2AW, Connector_Molex:Molex_Mini-Fit_Jr_5569-04A2_2x02_P4.20mm_Horizontal, F.Cu at (114.0, 139.4)
- added J13: BOOMELE 4.2-2*2AW, Connector_Molex:Molex_Mini-Fit_Jr_5569-04A2_2x02_P4.20mm_Horizontal, F.Cu at (102.4, 139.4)
- added J14: BOOMELE 4.2-2*3AW, Connector_Molex:Molex_Mini-Fit_Jr_5569-06A2_2x03_P4.20mm_Horizontal, F.Cu at (158.5, 138.9)
- added J15: BOOMELE 4.2-2*3AW, Connector_Molex:Molex_Mini-Fit_Jr_5569-06A2_2x03_P4.20mm_Horizontal, F.Cu at (142.6, 138.9)
- added J16: BOOMELE 4.2-2*4AW, Connector_Molex:Molex_Mini-Fit_Jr_5569-08A2_2x04_P4.20mm_Horizontal, F.Cu at (181.3, 44.8)
- added J17: BOOMELE 4.2-2*2AW, Connector_Molex:Molex_Mini-Fit_Jr_5569-04A2_2x02_P4.20mm_Horizontal, F.Cu at (90.8, 139.4)
- added J18: BOOMELE 4.2-2*2AW, Connector_Molex:Molex_Mini-Fit_Jr_5569-04A2_2x02_P4.20mm_Horizontal, F.Cu at (79.1, 139.4)
- added J19: BOOMELE 4.2-2*2AW, Connector_Molex:Molex_Mini-Fit_Jr_5569-04A2_2x02_P4.20mm_Horizontal, F.Cu at (67.5, 139.4)
- added J2: BOOMELE 4.2-2*3AW, Connector_Molex:Molex_Mini-Fit_Jr_5569-06A2_2x03_P4.20mm_Horizontal, F.Cu at (221.9, 138.9)
- added J3: BOOMELE 4.2-2*3AW, Connector_Molex:Molex_Mini-Fit_Jr_5569-06A2_2x03_P4.20mm_Horizontal, F.Cu at (206.0, 138.9)
- added J4: BOOMELE 4.2-2*3AW, Connector_Molex:Molex_Mini-Fit_Jr_5569-06A2_2x03_P4.20mm_Horizontal, F.Cu at (190.2, 138.9)
- added J5: BOOMELE 4.2-2*3AW, Connector_Molex:Molex_Mini-Fit_Jr_5569-06A2_2x03_P4.20mm_Horizontal, F.Cu at (174.3, 138.9)
- added J6: BOOMELE 4.2-2*4AW, Connector_Molex:Molex_Mini-Fit_Jr_5569-08A2_2x04_P4.20mm_Horizontal, F.Cu at (81.1, 44.8)
- added J7: BOOMELE 4.2-2*4AW, Connector_Molex:Molex_Mini-Fit_Jr_5569-08A2_2x04_P4.20mm_Horizontal, F.Cu at (101.2, 44.8)
- added J8: BOOMELE 4.2-2*4AW, Connector_Molex:Molex_Mini-Fit_Jr_5569-08A2_2x04_P4.20mm_Horizontal, F.Cu at (121.2, 44.8)
- added J9: BOOMELE 4.2-2*4AW, Connector_Molex:Molex_Mini-Fit_Jr_5569-08A2_2x04_P4.20mm_Horizontal, F.Cu at (141.2, 44.8)
- added L1: PSPMAA1050H-560M-ANP, Inductor_SMD:L_Sunlord_MWSA1005S, F.Cu at (105.4, 85.7)
- added R1: 47Ω 75V, Resistor_SMD:R_0603_1608Metric, F.Cu at (131.7, 93.6)
- added R2: 47Ω 75V, Resistor_SMD:R_0603_1608Metric, F.Cu at (131.7, 96.2)
- added R3: 100K 75V, Resistor_SMD:R_0603_1608Metric, F.Cu at (125.6, 107.7)
- added R4: 23.7kΩ 200V, Resistor_SMD:R_1206_3216Metric, F.Cu at (115.2, 93.1)
- added R5: 453kΩ 200V, Resistor_SMD:R_1206_3216Metric, F.Cu at (115.2, 96.4)
- added R6: 453kΩ 200V, Resistor_SMD:R_1206_3216Metric, F.Cu at (115.2, 99.8)
- added R7: 47kΩ, Resistor_SMD:R_0805_2012Metric, F.Cu at (115.1, 87.9)
- added R8: 2.8MΩ, Resistor_SMD:R_1206_3216Metric, F.Cu at (115.2, 103.1)
- added R9: 100KΩ, Resistor_SMD:R_1206_3216Metric, F.Cu at (115.2, 106.4)
- added U1: NAU7802SGI, Package_SO:SOIC-16_3.9x9.9mm_P1.27mm, F.Cu at (138.0, 85.7)
- added U2: LM5012QDDARQ1, Package_SO:SOIC-8-1EP_3.9x4.9mm_P1.27mm_EP2.95x4.9mm_Mask2.71x3.4mm_ThermalVias, F.Cu at (117.2, 83.2)

Commit message: ADD: Fuente de 24V a 5V para los Lidar
Other:
- copper layers 4 -> 2
- board text added: "Max Dim: 170x300mm"
Changed lines of the file:
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@@
 	(generator_version "9.0")
 	(general
-		(thickness 1.6002)
+		(thickness 1.6)
 		(legacy_teardrops no)
 	)
@@
 	)
 	(layers
-		(0 "F.Cu" signal "Front")
-		(4 "In1.Cu" signal)
-		(6 "In2.Cu" signal)
-		(2 "B.Cu" signal "Back")
+		(0 "F.Cu" signal)
+		(2 "B.Cu" signal)
+		(9 "F.Adhes" user "F.Adhesive")
+		(11 "B.Adhes" user "B.Adhesive")
 		(13 "F.Paste" user)
 		(15 "B.Paste" user)
@@
 		(1 "F.Mask" user)
 		(3 "B.Mask" user)
+		(17 "Dwgs.User" user "User.Drawings")
+		(19 "Cmts.User" user "User.Comments")
+		(21 "Eco1.User" user "User.Eco1")
+		(23 "Eco2.User" user "User.Eco2")
 		(25 "Edge.Cuts" user)
 		(27 "Margin" user)
@@
 		(29 "B.CrtYd" user "B.Courtyard")
 		(35 "F.Fab" user)
+		(33 "B.Fab" user)
+		(39 "User.1" user)
+		(41 "User.2" user)
+		(43 "User.3" user)
+		(45 "User.4" user)
 	)
 	(setup
+		(stackup
+			(layer "F.SilkS"
+				(type "Top Silk Screen")
+			)
+			(layer "F.Paste"
+				(type "Top Solder Paste")
+			)
+			(layer "F.Mask"
+				(type "Top Solder Mask")
+				(thickness 0.01)
+			)
+			(layer "F.Cu"
+				(type "copper")
+				(thickness 0.035)
+			)
+			(layer "dielectric 1"
+				(type "core")
+				(thickness 1.51)
+				(material "FR4")
+				(epsilon_r 4.5)
+				(loss_tangent 0.02)
+			)
+			(layer "B.Cu"
+				(type "copper")
+				(thickness 0.035)
+			)
+			(layer "B.Mask"
+				(type "Bottom Solder Mask")
+				(thickness 0.01)
+			)
+			(layer "B.Paste"
+				(type "Bottom Solder Paste")
+			)
+			(layer "B.SilkS"
+				(type "Bottom Silk Screen")
+			)
+			(copper_finish "None")
+			(dielectric_constraints no)
+		)
 		(pad_to_mask_clearance 0)
-		(solder_mask_min_width 0.12)
 		(allow_soldermask_bridges_in_footprints no)
 		(tenting front back)
@@
 		)
 	)
+	(gr_text "Max Dim: 170x300mm"
+		(at 23.75 192.25 0)
+		(layer "User.1")
+		(effects
+			(font
+				(size 4 4)
+				(thickness 0.5)
+			)
+			(justify left bottom)
+		)
+	)

Commit message: Primer sesion de ruteo
Parts:
- removed the J19 at (67.5, 139.4)
- added C16: 100nF 50V X7R, Capacitor_SMD:C_0603_1608Metric, F.Cu at (259.6, 336.0)
- added C17: 10uF 50V X7R, Capacitor_SMD:C_1206_3216Metric, F.Cu at (256.6, 326.5)
- added C18: 100nF 50V X7R, Capacitor_SMD:C_0603_1608Metric, F.Cu at (256.9, 328.8)
- added C19: 22uF 50V X7R, Capacitor_SMD:C_1812_4532Metric, F.Cu at (261.4, 326.8)
- added C20: 22uF 50V X7R, Capacitor_SMD:C_1812_4532Metric, F.Cu at (266.3, 326.8)
- added C21: 50V 75pF C0G, Capacitor_SMD:C_0603_1608Metric, F.Cu at (260.1, 342.0)
- added G***: LOGO, LOGO, F.Cu at (345.2, 290.7)
- added H1: MountingHole_Pad, MountingHole:MountingHole_3.2mm_M3_Pad_Via, F.Cu at (317.0, 72.0)
- added H2: MountingHole_Pad, MountingHole:MountingHole_3.2mm_M3_Pad_Via, F.Cu at (264.0, 184.0)
- added H3: MountingHole_Pad, MountingHole:MountingHole_3.2mm_M3_Pad_Via, F.Cu at (211.0, 72.0)
- added H4: MountingHole_Pad, MountingHole:MountingHole_3.2mm_M3_Pad_Via, F.Cu at (211.0, 387.0)
- added H5: MountingHole_Pad, MountingHole:MountingHole_3.2mm_M3_Pad_Via, F.Cu at (317.0, 387.0)
- added J11: BOOMELE 4.2-2*3AW, 0_ZA_Lib:Molex_Mini-Fit_Jr_5569-06A2_2x03_P4.20mm_Horizontal, F.Cu at (240.1, 376.9)
- added J15: BOOMELE 4.2-2*3AW, 0_ZA_Lib:Molex_Mini-Fit_Jr_5569-06A2_2x03_P4.20mm_Horizontal, F.Cu at (229.3, 149.2)
- added J2: BOOMELE 4.2-2*3AW, 0_ZA_Lib:Molex_Mini-Fit_Jr_5569-06A2_2x03_P4.20mm_Horizontal, F.Cu at (297.7, 161.1)
- added J21: BOOMELE 4.2-2*4AW, 0_ZA_Lib:Molex_Mini-Fit_Jr_5569-08A2_2x04_P4.20mm_Horizontal, F.Cu at (229.0, 170.3)
- added J23: BOOMELE 4.2-2*4AW, 0_ZA_Lib:Molex_Mini-Fit_Jr_5569-08A2_2x04_P4.20mm_Horizontal, F.Cu at (298.5, 123.9)
- added JP1: SolderJumper_2_Open, Jumper:SolderJumper-2_P1.3mm_Open_TrianglePad1.0x1.5mm, F.Cu at (271.5, 173.6)
- added JP2: SolderJumper_2_Open, Jumper:SolderJumper-2_P1.3mm_Open_TrianglePad1.0x1.5mm, F.Cu at (271.5, 170.2)
- added L2: cjiang FXL0630-150-M, Inductor_SMD:L_Sunlord_MWSA0624S, F.Cu at (264.1, 319.8)
- added R1: 2K2, Resistor_SMD:R_1206_3216Metric, F.Cu at (267.1, 173.6)
- added R13: 49.9Ω, Resistor_SMD:R_1206_3216Metric, F.Cu at (264.9, 339.2)
- added R14: 100KΩ, Resistor_SMD:R_1206_3216Metric, F.Cu at (259.9, 339.2)
- added R15: 13.3KΩ, Resistor_SMD:R_1206_3216Metric, F.Cu at (254.9, 339.2)
- added R2: 2K2, Resistor_SMD:R_1206_3216Metric, F.Cu at (267.1, 170.2)
- added U3: TPS54202DDC, Package_TO_SOT_SMD:SOT-23-6, F.Cu at (256.9, 333.5)
- F1: value Fuse -> Panel Solar Fuse 10x38
- J10: renamed from J13; footprint Connector_Molex:Molex_Mini-Fit_Jr_5569-04A2_2x02_P4.20mm_Horizontal -> 0_ZA_Lib:Molex_Mini-Fit_Jr_5569-04A2_2x02_P4.20mm_Horizontal
- J12: renamed from J7; footprint Connector_Molex:Molex_Mini-Fit_Jr_5569-08A2_2x04_P4.20mm_Horizontal -> 0_ZA_Lib:Molex_Mini-Fit_Jr_5569-08A2_2x04_P4.20mm_Horizontal
- J13: renamed from J8; footprint Connector_Molex:Molex_Mini-Fit_Jr_5569-08A2_2x04_P4.20mm_Horizontal -> 0_ZA_Lib:Molex_Mini-Fit_Jr_5569-08A2_2x04_P4.20mm_Horizontal
- J14: footprint Connector_Molex:Molex_Mini-Fit_Jr_5569-06A2_2x03_P4.20mm_Horizontal -> 0_ZA_Lib:Molex_Mini-Fit_Jr_5569-06A2_2x03_P4.20mm_Horizontal
- J16: renamed from J9; footprint Connector_Molex:Molex_Mini-Fit_Jr_5569-08A2_2x04_P4.20mm_Horizontal -> 0_ZA_Lib:Molex_Mini-Fit_Jr_5569-08A2_2x04_P4.20mm_Horizontal
- J17: renamed from J10; footprint Connector_Molex:Molex_Mini-Fit_Jr_5569-08A2_2x04_P4.20mm_Horizontal -> 0_ZA_Lib:Molex_Mini-Fit_Jr_5569-08A2_2x04_P4.20mm_Horizontal
- J18: renamed from J15; footprint Connector_Molex:Molex_Mini-Fit_Jr_5569-06A2_2x03_P4.20mm_Horizontal -> 0_ZA_Lib:Molex_Mini-Fit_Jr_5569-06A2_2x03_P4.20mm_Horizontal
- J19: renamed from J17; footprint Connector_Molex:Molex_Mini-Fit_Jr_5569-04A2_2x02_P4.20mm_Horizontal -> 0_ZA_Lib:Molex_Mini-Fit_Jr_5569-04A2_2x02_P4.20mm_Horizontal
- J20: renamed from J16; footprint Connector_Molex:Molex_Mini-Fit_Jr_5569-08A2_2x04_P4.20mm_Horizontal -> 0_ZA_Lib:Molex_Mini-Fit_Jr_5569-08A2_2x04_P4.20mm_Horizontal
- J22: renamed from J18; footprint Connector_Molex:Molex_Mini-Fit_Jr_5569-04A2_2x02_P4.20mm_Horizontal -> 0_ZA_Lib:Molex_Mini-Fit_Jr_5569-04A2_2x02_P4.20mm_Horizontal
- J3: renamed from J6; footprint Connector_Molex:Molex_Mini-Fit_Jr_5569-08A2_2x04_P4.20mm_Horizontal -> 0_ZA_Lib:Molex_Mini-Fit_Jr_5569-08A2_2x04_P4.20mm_Horizontal
- J4: renamed from J2; footprint Connector_Molex:Molex_Mini-Fit_Jr_5569-06A2_2x03_P4.20mm_Horizontal -> 0_ZA_Lib:Molex_Mini-Fit_Jr_5569-06A2_2x03_P4.20mm_Horizontal
- J5: renamed from J3; footprint Connector_Molex:Molex_Mini-Fit_Jr_5569-06A2_2x03_P4.20mm_Horizontal -> 0_ZA_Lib:Molex_Mini-Fit_Jr_5569-06A2_2x03_P4.20mm_Horizontal
- J6: renamed from J11; footprint Connector_Molex:Molex_Mini-Fit_Jr_5569-24A2_2x12_P4.20mm_Horizontal -> 0_ZA_Lib:Molex_Mini-Fit_Jr_5569-24A2_2x12_P4.20mm_Horizontal
- J7: renamed from J4; footprint Connector_Molex:Molex_Mini-Fit_Jr_5569-06A2_2x03_P4.20mm_Horizontal -> 0_ZA_Lib:Molex_Mini-Fit_Jr_5569-06A2_2x03_P4.20mm_Horizontal
- J8: renamed from J5; footprint Connector_Molex:Molex_Mini-Fit_Jr_5569-06A2_2x03_P4.20mm_Horizontal -> 0_ZA_Lib:Molex_Mini-Fit_Jr_5569-06A2_2x03_P4.20mm_Horizontal
- J9: renamed from J12; footprint Connector_Molex:Molex_Mini-Fit_Jr_5569-04A2_2x02_P4.20mm_Horizontal -> 0_ZA_Lib:Molex_Mini-Fit_Jr_5569-04A2_2x02_P4.20mm_Horizontal
- moved J16 333.9 mm to (297.5, 339.8), turned to -90 degrees
- moved J17 315.0 mm to (229.3, 352.3), turned to 90 degrees
- moved J6 269.9 mm to (294.1, 376.7), turned to 180 degrees
- moved L1 266.9 mm to (264.0, 300.3), turned to -90 degrees
- moved J22 266.7 mm to (298.0, 291.8), turned to -90 degrees
- moved J1 265.0 mm to (285.8, 232.8), turned to -90 degrees
- moved J3 264.2 mm to (298.0, 195.6), turned to -90 degrees
- moved C13 260.0 mm to (264.2, 311.5)
- moved R9 252.7 mm to (256.5, 297.3), turned to 180 degrees
- moved C11 252.5 mm to (255.3, 308.0)
- moved U2 247.7 mm to (257.9, 287.0), turned to -90 degrees
- moved D1 246.2 mm to (263.8, 287.0)
- moved C12 244.7 mm to (255.3, 303.8)
- moved R6 243.4 mm to (256.3, 294.8)
- moved J10 239.5 mm to (298.7, 276.6), turned to -90 degrees
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- renumbered C4 to C1, C12 to C11, C13 to C12, C11 to C13, C15 to C14, C14 to C15, C3 to C2, C1 to C3, C2 to C4, R9 to R10, R4 to R11, R1 to R3, R2 to R4, R3 to R5, R5 to R6, R6 to R7, R7 to R9
Connections:
- net /LIDAR_1_RX_SCL renamed /LIDAR_1_TX
- net /LIDAR_2_RX_SCL renamed /LIDAR_2_TX
- net /PWM_Asp_BR renamed /CAN_B_-_9
- C1 pad 1: Net-(U1-DVDD) -> +3V3
- J1 pad 3: /CAN_H_1 -> /CAN_B_+_2
- J1 pad 4: /CAN_L_1 -> /CAN_B_-_2
- J1 pad 5: unconnected-(J1-Pin_5-Pad5) -> /CAN_B_+_1
- J1 pad 6: unconnected-(J1-Pin_6-Pad6) -> /CAN_B_-_1
- J10 pad 2: GND -> /PWM_Light
- J10 pad 3: /PWM_Light -> GND
- J12 pad 1: GND -> /CAN_B_+_5
- J12 pad 2: /PWM_Asp_FR -> /CAN_B_-_5
- J12 pad 3: /CAN_H_6 -> /CAN_B_-_4
- J12 pad 4: /CAN_L_6 -> /CAN_B_+_4
- J12 pad 5: /CAN_H_7 -> unconnected-(J12-Pin_5-Pad5)
- J12 pad 6: /CAN_L_7 -> GND
- J13 pad 1: GND -> /CAN_B_+_6
- J13 pad 2: /PWM_Asp_FL -> /CAN_B_-_6
- J13 pad 3: /CAN_H_7 -> /CAN_B_-_5
- J13 pad 4: /CAN_L_7 -> /CAN_B_+_5
- J13 pad 5: /CAN_H_8 -> unconnected-(J13-Pin_5-Pad5)
- J13 pad 6: /CAN_L_8 -> GND
- J14 pad 4: /LIDAR_1_TX_SDA -> /I2C_DAT
- J14 pad 5: GND -> /I2C_CLK
- J14 pad 6: unconnected-(J14-Pin_6-Pad6) -> /LIDAR_1_RX
- J16 pad 1: GND -> /CAN_B_+_9
- J16 pad 3: /CAN_H_8 -> /CAN_B_-_8
- J16 pad 4: /CAN_L_8 -> /CAN_B_+_8
- J16 pad 5: /CAN_H_9 -> unconnected-(J16-Pin_5-Pad5)
- J16 pad 6: /CAN_L_9 -> GND
- J17 pad 1: GND -> /CAN_B_+_7
- J17 pad 2: /PWM_Asp_BL -> /CAN_B_-_7
- J17 pad 3: /CAN_H_9 -> /CAN_B_-_6
- J17 pad 4: /CAN_L_9 -> /CAN_B_+_6
- J17 pad 5: /CAN_H_10 -> unconnected-(J17-Pin_5-Pad5)
- J17 pad 6: /CAN_L_10 -> GND
- J18 pad 4: /LIDAR_2_TX_SDA -> /I2C_DAT
- J18 pad 5: GND -> /I2C_CLK
- J18 pad 6: unconnected-(J15-Pin_6-Pad6) -> /LIDAR_2_RX
- J22 pad 3: /FLOW_OUT_SIGNAL -> unconnected-(J22-Pin_3-Pad3)
- J22 pad 4: unconnected-(J18-Pin_4-Pad4) -> /FLOW_OUT_SIGNAL
- J3 pad 1: GND -> /CAN_B_+_3
- J3 pad 2: /PWM_Pump -> /CAN_B_-_3
- J3 pad 3: /CAN_H_5 -> /CAN_B_-_2
- J3 pad 4: /CAN_L_5 -> /CAN_B_+_2
- J3 pad 5: /CAN_H_6 -> unconnected-(J3-Pin_5-Pad5)
- J3 pad 6: /CAN_L_6 -> GND
- J4 pad 1: /CAN_H_1 -> /CAN_A_-_3
- J4 pad 2: /CAN_L_1 -> /CAN_A_-_2
- J4 pad 3: /CAN_H_2 -> /CAN_A_+_2
- J4 pad 4: /CAN_L_2 -> /CAN_A_+_3
- J5 pad 1: /CAN_H_2 -> /CAN_A_-_4
- J5 pad 2: /CAN_L_2 -> /CAN_A_-_3
- J5 pad 3: /CAN_H_3 -> /CAN_A_+_3
- J5 pad 4: /CAN_L_3 -> /CAN_A_+_4
- J6 pad 1: unconnected-(J11-Pin_1-Pad1) -> /CAN_A_-_1
- J6 pad 10: unconnected-(J11-Pin_10-Pad10) -> /EXTRA_2
- J6 pad 11: unconnected-(J11-Pin_11-Pad11) -> +24V
- J6 pad 12: unconnected-(J11-Pin_12-Pad12) -> /I2C_CLK
- J6 pad 13: unconnected-(J11-Pin_13-Pad13) -> /CAN_A_+_1
- J6 pad 14: unconnected-(J11-Pin_14-Pad14) -> /CAN_B_+_8
- J6 pad 15: unconnected-(J11-Pin_15-Pad15) -> /PWM_Mot_FR
- J6 pad 16: unconnected-(J11-Pin_16-Pad16) -> /FLOW_OUT_SIGNAL
- J6 pad 17: unconnected-(J11-Pin_17-Pad17) -> GND
- J6 pad 18: unconnected-(J11-Pin_18-Pad18) -> /EQEP_A
- J6 pad 19: unconnected-(J11-Pin_19-Pad19) -> +3V3
- J6 pad 2: unconnected-(J11-Pin_2-Pad2) -> /CAN_B_-_8
- J6 pad 20: unconnected-(J11-Pin_20-Pad20) -> /LC_DRDY
- J6 pad 21: unconnected-(J11-Pin_21-Pad21) -> GND
- J6 pad 22: unconnected-(J11-Pin_22-Pad22) -> GND
- J6 pad 23: unconnected-(J11-Pin_23-Pad23) -> +24V
- J6 pad 24: unconnected-(J11-Pin_24-Pad24) -> /I2C_DAT
- J6 pad 3: unconnected-(J11-Pin_3-Pad3) -> /PWM_Mot_BR
- J6 pad 4: unconnected-(J11-Pin_4-Pad4) -> /PWM_Light
- J6 pad 5: unconnected-(J11-Pin_5-Pad5) -> /EXTRA_3
- J6 pad 6: unconnected-(J11-Pin_6-Pad6) -> /EXTRA_1
- J6 pad 9: unconnected-(J11-Pin_9-Pad9) -> /EQEP_I
- J7 pad 1: /CAN_H_3 -> /CAN_A_-_2
- J7 pad 2: /CAN_L_3 -> /CAN_A_-_1
- J7 pad 3: /CAN_H_4 -> /CAN_A_+_1
- J7 pad 4: /CAN_L_4 -> /CAN_A_+_2
- J8 pad 1: /CAN_H_4 -> /CAN_A_-_5
- J8 pad 2: /CAN_L_4 -> /CAN_A_-_4
- J8 pad 3: /CAN_H_5 -> /CAN_A_+_4
- J8 pad 4: /CAN_L_5 -> /CAN_A_+_5
- J9 pad 2: GND -> /PWM_Light
- J9 pad 3: /PWM_Light -> GND
- U1 pad 13: /LC_SCLK -> /I2C_CLK
- U1 pad 14: /LC_SDIO -> /I2C_DAT
- U1 pad 15: Net-(U1-DVDD) -> +3V3
- U2 pad 9: unconnected-(U2-EP-Pad9) -> GND
Routing:
- net /VBat: track 0.00 -> 856.9 mm
- net +5V: track 0.00 -> 608.7 mm, vias 0 -> 2
- net +24V: track 0.00 -> 526.5 mm, vias 0 -> 6
- net /I2C_CLK: track 0.00 -> 411.4 mm, vias 0 -> 4
- net /I2C_DAT: track 0.00 -> 399.4 mm, vias 0 -> 1
- net /CAMERA_TX: track 0.00 -> 363.0 mm, vias 0 -> 11
- net /CAMERA_RX: track 0.00 -> 347.4 mm, vias 0 -> 11
- net /PWM_Mot_FL: track 0.00 -> 339.1 mm, vias 0 -> 8
- net /PWM_Mot_FR: track 0.00 -> 326.1 mm, vias 0 -> 12
- net /CAN_A_+_4: track 0.00 -> 270.2 mm, vias 0 -> 2
- net /CAN_A_-_4: track 0.00 -> 265.2 mm, vias 0 -> 2
- net /CAN_A_+_2: track 0.00 -> 263.2 mm, vias 0 -> 6
- net /CAN_B_-_6: track 0.00 -> 261.0 mm, vias 0 -> 4
- net /CAN_B_+_6: track 0.00 -> 259.3 mm, vias 0 -> 4
- net /CAN_A_-_2: track 0.00 -> 258.9 mm, vias 0 -> 6
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- added copper zone on F.Cu, net +24V
- added copper zone on F.Cu, net +5V
- added copper zone on F.Cu, net GND
- added copper zone on F.Cu, net Net-(D1-K)
- added copper zone on F.Cu, net Net-(U2-FB)
- added copper zone on F.Cu, net Net-(U3-SW)
Other:
- board outline added: 116 x 325 mm
- board text added: "BATT"
- board text added: "CAMERA"
- board text added: "EXTRA"
- board text added: "FLOW"
- board text added: "LIDAR1"
- board text added: "LIDAR2"
- board text added: "LIDAR3"
- board text added: "LIGHT1"
- board text added: "LIGHT2"
- board text added: "LOADCELL"
- board text added: "M1 A1"
- board text added: "M2 A2"
- board text added: "M3 A3"
- board text added: "M4 A4"
- board text added: "MEX"
- board text added: "Max Dim: 136mmx400mmx60mm"
- board text added: "PUMP"
- board text added: "Panel Solar Fuse 10x38"
- board text added: "VERONTE"
- board text added: "pDDL"
- board text removed: "Max Dim: 170x300mm"

Commit message: Agregado los testpoint, falta leds indicadores y serigrafia y cerramos
Parts:
- added TP1: +BATT, 0_ZA_Lib:TestPoint_Pad_D2.0mm_silk_value, F.Cu at (283.0, 251.8)
- added TP12: CAM_RX, 0_ZA_Lib:TestPoint_Pad_D2.0mm_silk_value, F.Cu at (229.2, 81.0)
- added TP13: CAM_TX, 0_ZA_Lib:TestPoint_Pad_D2.0mm_silk_value, F.Cu at (236.8, 81.0)
- added TP14: PWM_MOT_FR, 0_ZA_Lib:TestPoint_Pad_D2.0mm_silk_value, F.Cu at (308.0, 97.5)
- added TP15: PWM_MOT_BR, 0_ZA_Lib:TestPoint_Pad_D2.0mm_silk_value, F.Cu at (315.8, 318.0)
- added TP16: PWM_MOT_BL, 0_ZA_Lib:TestPoint_Pad_D2.0mm_silk_value, F.Cu at (220.5, 318.5)
- added TP17: PWM_MOT_FL, 0_ZA_Lib:TestPoint_Pad_D2.0mm_silk_value, F.Cu at (216.0, 120.8)
- added TP18: FLOW_S, 0_ZA_Lib:TestPoint_Pad_D2.0mm_silk_value, F.Cu at (301.5, 302.2)
- added TP19: PWM_LIGHT, 0_ZA_Lib:TestPoint_Pad_D2.0mm_silk_value, F.Cu at (298.7, 286.2)
- added TP2: VBat, 0_ZA_Lib:TestPoint_Pad_D2.0mm_silk_value, F.Cu at (279.0, 213.7)
- added TP20: +24V, 0_ZA_Lib:TestPoint_Pad_D2.0mm_silk_value, F.Cu at (289.2, 311.5)
- added TP21: +5V, 0_ZA_Lib:TestPoint_Pad_D2.0mm_silk_value, F.Cu at (294.2, 311.5)
- added TP22: +3V3, 0_ZA_Lib:TestPoint_Pad_D2.0mm_silk_value, F.Cu at (298.8, 311.5)
- added TP23: I2C_DAT, 0_ZA_Lib:TestPoint_Pad_D2.0mm_silk_value, F.Cu at (265.5, 259.4)
- added TP24: I2C_CLK, 0_ZA_Lib:TestPoint_Pad_D2.0mm_silk_value, F.Cu at (265.5, 263.5)
- added TP25: FB_24V, 0_ZA_Lib:TestPoint_Pad_D2.0mm_silk_value, F.Cu at (249.0, 289.8)
- added TP26: FB_5V, 0_ZA_Lib:TestPoint_Pad_D2.0mm_silk_value, F.Cu at (253.2, 335.0)
- added TP27: LC_DRDY, 0_ZA_Lib:TestPoint_Pad_D2.0mm_silk_value, F.Cu at (308.8, 175.0)
- added TP28: CAN_B_-_3, 0_ZA_Lib:TestPoint_Pad_D2.0mm_silk_value, F.Cu at (302.5, 190.8)
- added TP29: CAN_B_+_3, 0_ZA_Lib:TestPoint_Pad_D2.0mm_silk_value, F.Cu at (298.5, 190.8)
- added TP3: GND, 0_ZA_Lib:TestPoint_Pad_D2.0mm_silk_value, F.Cu at (283.5, 311.5)
- added TP4: CAN_B_+_1, 0_ZA_Lib:TestPoint_Pad_D2.0mm_silk_value, F.Cu at (299.5, 252.5)
- added TP5: CAN_B_-_1, 0_ZA_Lib:TestPoint_Pad_D2.0mm_silk_value, F.Cu at (303.5, 252.5)
- added TP8: CAN_B_+_7, 0_ZA_Lib:TestPoint_Pad_D2.0mm_silk_value, F.Cu at (223.5, 358.6)
- added TP9: CAN_B_-_7, 0_ZA_Lib:TestPoint_Pad_D2.0mm_silk_value, F.Cu at (227.6, 358.6)
- U2: footprint Package_SO:SOIC-8-1EP_3.9x4.9mm_P1.27mm_EP2.95x4.9mm_Mask2.71x3.4mm_ThermalVias -> 0_ZA_Lib:SOIC-8-1EP_3.9x4.9mm_P1.27mm_EP2.95x4.9mm_Mask2.71x3.4mm_ThermalVias
- moved G*** 130.4 mm to (232.5, 225.1)
Connections:
- J21 pad 2: /EXTRA_1 -> GND
- J21 pad 3: /EQEP_I -> unconnected-(J21-Pin_3-Pad3)
- J21 pad 5: unconnected-(J21-Pin_5-Pad5) -> /EQEP_I
- J21 pad 6: GND -> /EXTRA_2
- J21 pad 7: /EXTRA_2 -> /EXTRA_1
- J6 pad 10: /EXTRA_2 -> /EXTRA_1
- J6 pad 17: GND -> +3V3
- J6 pad 18: /EQEP_A -> GND
- J6 pad 19: +3V3 -> GND
- J6 pad 20: /LC_DRDY -> unconnected-(J6-Pin_20-Pad20)
- J6 pad 21: GND -> /EQEP_A
- J6 pad 22: GND -> /EXTRA_3
- J6 pad 5: /EXTRA_3 -> GND
- J6 pad 6: /EXTRA_1 -> /LC_DRDY
- J6 pad 8: unconnected-(J6-Pin_8-Pad8) -> /EQEP_I
- J6 pad 9: /EQEP_I -> /EXTRA_2
Routing:
- net /LC_DRDY: track 0.00 -> 299.2 mm, vias 0 -> 14
- net /EQEP_A: track 0.00 -> 263.3 mm, vias 0 -> 2
- net +3V3: track 21.4 -> 284.2 mm, vias 0 -> 15
- net /EXTRA_2: track 0.00 -> 258.0 mm
- net /EQEP_I: track 0.00 -> 257.1 mm
- net /EXTRA_1: track 0.00 -> 256.8 mm
- net /EXTRA_3: track 0.00 -> 249.9 mm, vias 0 -> 2
- net /VBat: track 856.9 -> 920.2 mm, vias 0 -> 2
- net /CAN_B_+_1: track 0.00 -> 32.8 mm
- net /PWM_Mot_BL: track 88.1 -> 117.5 mm
- net +24V: track 526.5 -> 554.8 mm, vias 6 -> 12
- net /CAN_B_-_1: track 0.00 -> 27.9 mm
- net /CAN_B_-_7: track 63.2 -> 77.6 mm, vias 0 -> 1
- net /CAN_B_-_3: track 91.6 -> 104.2 mm, vias 2 -> 3
- net +BATT: track 23.7 -> 33.7 mm
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- added copper zone on B.Cu, net +24V
- added copper zone on B.Cu, net +5V
- added copper zone on B.Cu, net GND
- added copper zone on B.Cu, net Net-(U3-SW)
Other:
- outline, holes or cut-outs redrawn
- board text added: "+"
- board text added: "-"
- board text added: "CAN_B_1"
- board text added: "CAN_B_3"
- board text added: "CAN_B_7"
